File: tof-sensor-board.sch (KiCad schematic (older format))
At the start: 39 parts, among them IC1 TLV710, U1 STM32F042C6T6, U2 LTC2875, U3 VL6180X, X1 16MHz

Commit message: change STM32F3 QFN32
Parts:
- removed C3: 0.1uF, Capacitors_SMD:C_0402, symbol C_Small
- removed C5: 1uF, Capacitors_SMD:C_0402, symbol C
- removed C6: 0.01uF, Capacitors_SMD:C_0402, symbol C
- removed C7: 0.1uF, Capacitors_SMD:C_0402, symbol C
- removed CONN1: SWD, _connectors:_SoldarPad2mm_5, symbol SWD
- removed D1: POWER, _std:_0603, symbol LED
- removed R1: 100k, Resistors_SMD:R_0402, symbol R_Small
- removed R2: 100k, Resistors_SMD:R_0402, symbol R
- removed R5: 1k, Resistors_SMD:R_0402, symbol R
- removed U1: STM32F042C6T6, _lqfp:_LQFP48, symbol STM32F042C6T6
- added C3: 0.1uF, symbol C
- added CONN1: SWD/DEBUG, MODULE, symbol SWD/DEBUG
- added U?: STM32F302K8U6, MODULE, symbol STM32F302K8U6
Connections:
- net labels added: STM32_NRST, STM32_SWCLK, STM32_SWDIO, UART2_RX, UART2_TX
- net labels removed: STM32F0_NRST, STM32F0_SWCLK, STM32F0_SWDIO
- wire segments 125 -> 129
- no-connect marks 29 -> 14
Other:
- moved on the sheet: C1, C2, C4, C8, C9, R3, R4, X1
